Commit message: V1.0.1-修改部分代码以适配noetic版本

File: urdf/diff_wheeled_robot.xacro (robot description, xacro)
@@ -80,5 +80,5 @@
       <origin xyz="0 0 0" />
       <!--The 3x3 rotational inertia matrix. -->
-        <cylinder_inertia  m="${base_mass}" r="${base_radius}" h="${base_height}" />
+      <xacro:cylinder_inertia  m="${base_mass}" r="${base_radius}" h="${base_height}" />
     </inertial>
     <visual>

File: urdf/pan_tilt_generated.urdf (robot description, URDF)
Before this commit: robot pan_tilt, 3 links, 2 joints
Links:
- link tilt_link: geometry collision cylinder length=0.4 radius=0.24000000000000002; visual cylinder length=0.4 radius=0.04
